Commit message: Renamed package to "rtabmap_drone_example". Updated config files for PX4 v1.12.3. Added new world "apt". Reduced drone size to pass doorways. Improved texture of "room" world. Updated rviz config. Connected rtabmap goal interface to move_base.

File: urdf/drone.urdf.xacro (robot description, xacro)
@@ -1,9 +1,10 @@
 <?xml version="1.0"?>
 <robot xmlns:xacro="http://www.ros.org/wiki/xacro" name="iris">
-  <xacro:include filename="$(find mavros_nav_2d)/urdf/drone.gazebo"/>
+  <xacro:include filename="$(find rtabmap_drone_example)/urdf/drone.gazebo"/>
+  <xacro:property name="scale" value="0.75" />
    <link name='base_link'>
       <inertial>
         <origin xyz="0 0 0" rpy="0 0 0"/>
-        <mass value="1.5"/>
+        <mass value="${1.5 * scale}"/>
         <inertia
 	  ixx="0.0347563" ixy="0.0" ixz="0.0"
@@ -14,5 +15,5 @@
         <origin xyz="0 0 0" rpy="0 0 0"/>
         <geometry>
-          <box size="0.47 0.47 0.11"/>
+          <box size="${0.47*scale} ${0.47*scale} ${0.11*scale}"/>
         </geometry>
         <!--surface>
@@ -31,5 +32,5 @@
         <origin xyz="0 0 0" rpy="0 0 0"/>
         <geometry>
-          <mesh filename="package://mavlink_sitl_gazebo/models/rotors_description/meshes/iris.stl"/>
+          <mesh scale="${scale} ${scale} ${scale}" filename="package://mavlink_sitl_gazebo/models/iris/meshes/iris.stl"/>
         </geometry>
         <!--material name="base_link_material">
@@ -86,5 +87,5 @@
         <origin xyz="0 0 0" rpy="0 0 0"/>
         <geometry>
-          <mesh filename="package://mavlink_sitl_gazebo/models/rotors_description/meshes/iris_prop_ccw.dae"/>
+          <mesh scale="${scale} ${scale} ${scale}" filename="package://mavlink_sitl_gazebo/models/iris/meshes/iris_prop_ccw.dae"/>
         </geometry>
         <!-- material>
@@ -101,5 +102,5 @@
       <parent link="base_link"/>
       <child link="rotor_0"/>
-      <origin xyz="0.13 -0.22 0.023" rpy="0 0 0"/>
+      <origin xyz="${scale*0.13} ${scale*-0.22} ${scale*0.023}" rpy="0 0 0"/>
       <axis xyz="0 0 1"/>
       <limit lower="-1e+16" upper="1e+16" effort="0" velocity="0"/>
@@ -131,5 +132,5 @@
         <origin xyz="0 0 0" rpy="0 0 0"/>
         <geometry>
-          <mesh filename="package://mavlink_sitl_gazebo/models/rotors_description/meshes/iris_prop_ccw.dae"/>
+          <mesh scale="${scale} ${scale} ${scale}" filename="package://mavlink_sitl_gazebo/models/iris/meshes/iris_prop_ccw.dae"/>
         </geometry>
         <!-- material>
@@ -146,5 +147,5 @@
       <parent link="base_link"/>
       <child link="rotor_1"/>
-      <origin xyz="-0.13 0.2 0.023" rpy="0 0 0"/>
+      <origin xyz="${scale*-0.13} ${scale*0.2} ${scale*0.023}" rpy="0 0 0"/>
       <axis xyz="0 0 1"/>
       <limit lower="-1e+16" upper="1e+16" effort="0" velocity="0"/>
@@ -176,5 +177,5 @@
         <origin xyz="0 0 0" rpy="0 0 0"/>
         <geometry>
-          <mesh filename="package://mavlink_sitl_gazebo/models/rotors_description/meshes/iris_prop_cw.dae"/>
+          <mesh scale="${scale} ${scale} ${scale}" filename="package://mavlink_sitl_gazebo/models/iris/meshes/iris_prop_cw.dae"/>
         </geometry>
         <!-- material>
@@ -191,5 +192,5 @@
       <parent link="base_link"/>
       <child link="rotor_2"/>
-      <origin xyz="0.13 0.22 0.023" rpy="0 0 0"/>
+      <origin xyz="${scale*0.13} ${scale*0.22} ${scale*0.023}" rpy="0 0 0"/>
       <axis xyz="0 0 1"/>
       <limit lower="-1e+16" upper="1e+16" effort="0" velocity="0"/>
@@ -221,5 +222,5 @@
         <origin xyz="0 0 0" rpy="0 0 0"/>
         <geometry>
-          <mesh filename="package://mavlink_sitl_gazebo/models/rotors_description/meshes/iris_prop_cw.dae"/>
+          <mesh scale="${scale} ${scale} ${scale}" filename="package://mavlink_sitl_gazebo/models/iris/meshes/iris_prop_cw.dae"/>
         </geometry>
         <!-- material>
@@ -236,5 +237,5 @@
       <parent link="base_link"/>
       <child link="rotor_3"/>
-      <origin xyz="-0.13 -0.2 0.023" rpy="0 0 0"/>
+      <origin xyz="${scale*-0.13} ${scale*-0.2} ${scale*0.023}" rpy="0 0 0"/>
       <axis xyz="0 0 1"/>
       <limit lower="-1e+16" upper="1e+16" effort="0" velocity="0"/>
@@ -269,7 +270,7 @@
   </gazebo>
   <!-- Import macro for realsense-RS200 camera-->
-  <xacro:include filename="$(find mavros_nav_2d)/urdf/realsense-RS200.macro.xacro"/>
+  <xacro:include filename="$(find rtabmap_drone_example)/urdf/realsense-RS200.macro.xacro"/>
   <joint name="base_camera_joint" type="fixed">
-    <origin xyz="0.1 0 0" rpy="0 0 0" />
+    <origin xyz="${scale*0.1} 0 0" rpy="0 0 0" />
     <parent link="base_link"/>
     <child link="base_camera" />

Commit message: Fixed scale in rviz, Added robotmodel an 3d map in rviz

File: urdf/drone.urdf.xacro (robot description, xacro)
@@ -1,6 +1,7 @@
 <?xml version="1.0"?>
 <robot xmlns:xacro="http://www.ros.org/wiki/xacro" name="iris">
+  <xacro:arg name="scale" default="0.75"/>
+  <xacro:property name="scale" value="$(arg scale)" />
   <xacro:include filename="$(find rtabmap_drone_example)/urdf/drone.gazebo"/>
-  <xacro:property name="scale" value="0.75" />
    <link name='base_link'>
       <inertial>

Commit message: Updated parameters. Added landing/disarm with joystick.

File: urdf/drone.urdf.xacro (robot description, xacro)
@@ -9,7 +9,7 @@
         <mass value="${1.5 * scale}"/>
         <inertia
-	  ixx="0.0347563" ixy="0.0" ixz="0.0"
-	  iyy="0.0458929" iyz="0.0"
-	  izz="0.0977"/>
+	  ixx="${0.0347563 * scale}" ixy="0.0" ixz="0.0"
+	  iyy="${0.0458929 * scale}" iyz="0.0"
+	  izz="${0.0977 * scale}"/>
       </inertial>
       <collision>
@@ -65,5 +65,5 @@
       <inertial>
         <origin xyz="0 0 0" rpy="0 0 0"/>
-        <mass value="0.005"/>
+        <mass value="${0.005 * scale}"/>
         <inertia
 	  ixx="9.75e-07" ixy="0.0" ixz="0.0"
@@ -74,5 +74,5 @@
         <origin xyz="0 0 0" rpy="0 0 0"/>
         <geometry>
-          <cylinder length="0.005" radius="0.128"/>
+          <cylinder length="0.005" radius="${scale*0.128}"/>
         </geometry>
         <surface>
@@ -110,5 +110,5 @@
       <inertial>
         <origin xyz="0 0 0" rpy="0 0 0"/>
-        <mass value="0.005"/>
+        <mass value="${0.005 * scale}"/>
         <inertia
 	  ixx="9.75e-07" ixy="0.0" ixz="0.0"
@@ -119,5 +119,5 @@
         <origin xyz="0 0 0" rpy="0 0 0"/>
         <geometry>
-          <cylinder length="0.005" radius="0.128"/>
+          <cylinder length="0.005" radius="${scale*0.128}"/>
         </geometry>
         <surface>
@@ -155,5 +155,5 @@
       <inertial>
         <origin xyz="0 0 0" rpy="0 0 0"/>
-        <mass value="0.005"/>
+        <mass value="${0.005 * scale}"/>
         <inertia
 	  ixx="9.75e-07" ixy="0.0" ixz="0.0"
@@ -164,5 +164,5 @@
         <origin xyz="0 0 0" rpy="0 0 0"/>
         <geometry>
-          <cylinder length="0.005" radius="0.128"/>
+          <cylinder length="0.005" radius="${scale*0.128}"/>
         </geometry>
         <surface>
@@ -200,5 +200,5 @@
       <inertial>
         <origin xyz="0 0 0" rpy="0 0 0"/>
-        <mass value="0.005"/>
+        <mass value="${0.005 * scale}"/>
         <inertia
 	  ixx="9.75e-07" ixy="0.0" ixz="0.0"
@@ -209,5 +209,5 @@
         <origin xyz="0 0 0" rpy="0 0 0"/>
         <geometry>
-          <cylinder length="0.005" radius="0.128"/>
+          <cylinder length="0.005" radius="${scale*0.128}"/>
         </geometry>
         <surface>
@@ -250,5 +250,5 @@
      <inertial>
        <origin xyz="0 0 0" rpy="0 0 0"/>
-       <mass value="0.0000001"/>
+       <mass value="0.00001"/>
        <inertia
 	  ixx="1e-05" ixy="0.0" ixz="0.0"

Commit message: Backward compatibility with Melodic

File: urdf/drone.urdf.xacro (robot description, xacro)
@@ -2,5 +2,7 @@
 <robot xmlns:xacro="http://www.ros.org/wiki/xacro" name="iris">
   <xacro:arg name="scale" default="0.75"/>
+  <xacro:arg name="stl_path" default="mavlink_sitl_gazebo/models/iris/meshes"/>
   <xacro:property name="scale" value="$(arg scale)" />
+  <xacro:property name="stl_path" value="$(arg stl_path)" />
   <xacro:include filename="$(find rtabmap_drone_example)/urdf/drone.gazebo"/>
    <link name='base_link'>
@@ -33,5 +35,5 @@
         <origin xyz="0 0 0" rpy="0 0 0"/>
         <geometry>
-          <mesh scale="${scale} ${scale} ${scale}" filename="package://mavlink_sitl_gazebo/models/iris/meshes/iris.stl"/>
+          <mesh scale="${scale} ${scale} ${scale}" filename="package://${stl_path}/iris.stl"/>
         </geometry>
         <!--material name="base_link_material">
@@ -88,5 +90,5 @@
         <origin xyz="0 0 0" rpy="0 0 0"/>
         <geometry>
-          <mesh scale="${scale} ${scale} ${scale}" filename="package://mavlink_sitl_gazebo/models/iris/meshes/iris_prop_ccw.dae"/>
+          <mesh scale="${scale} ${scale} ${scale}" filename="package://${stl_path}/iris_prop_ccw.dae"/>
         </geometry>
         <!-- material>
@@ -133,5 +135,5 @@
         <origin xyz="0 0 0" rpy="0 0 0"/>
         <geometry>
-          <mesh scale="${scale} ${scale} ${scale}" filename="package://mavlink_sitl_gazebo/models/iris/meshes/iris_prop_ccw.dae"/>
+          <mesh scale="${scale} ${scale} ${scale}" filename="package://${stl_path}/iris_prop_ccw.dae"/>
         </geometry>
         <!-- material>
@@ -178,5 +180,5 @@
         <origin xyz="0 0 0" rpy="0 0 0"/>
         <geometry>
-          <mesh scale="${scale} ${scale} ${scale}" filename="package://mavlink_sitl_gazebo/models/iris/meshes/iris_prop_cw.dae"/>
+          <mesh scale="${scale} ${scale} ${scale}" filename="package://${stl_path}/iris_prop_cw.dae"/>
         </geometry>
         <!-- material>
@@ -223,5 +225,5 @@
         <origin xyz="0 0 0" rpy="0 0 0"/>
         <geometry>
-          <mesh scale="${scale} ${scale} ${scale}" filename="package://mavlink_sitl_gazebo/models/iris/meshes/iris_prop_cw.dae"/>
+          <mesh scale="${scale} ${scale} ${scale}" filename="package://${stl_path}/iris_prop_cw.dae"/>
         </geometry>
         <!-- material>
